File: LCD_HAT_pins_eink.kicad_pcb (KiCad board)
At the start: 4 copper layers, 45.7 x 80.4 mm, 33 parts, among them J1 Qwiic, J2 LCD, J3 PWR_JUMPER, J4 PWR_JUMPER, J5 AFC24-S24FIC-00, Q1 Si1308, SW1 SW_Push, SW2 SW_Push, U1 SeeeduinoXIAO

Commit message: Rework routing
Parts:
- removed J4: PWR_JUMPER, Connector_PinHeader_2.54mm:PinHeader_1x02_P2.54mm_Vertical
- moved R3 1.13 mm to (125.3, 84.2), turned to 135 degrees
- moved C4 0.50 mm to (152.2, 46.6)
- moved J1 0.22 mm to (136.8, 119.2)
Connections:
- J1 pad 2: Net-(J1-Pin_2) -> +3.3V
Routing:
- net SCL: track 12.2 -> 102.6 mm
- net Net-(A1-D0): track 16.3 -> 100.1 mm
- net Net-(A1-D1): track 4.12 -> 86.1 mm, vias 0 -> 1
- net SDA: track 44.2 -> 119.9 mm
- net /EPD_BUSY: track 61.2 -> 133.3 mm
- net /EPD_RST: track 51.2 -> 120.1 mm
- net /EPD_CLK: track 45.6 -> 103.4 mm
- net /EPD_CS: track 61.8 -> 114.4 mm, vias 1 -> 2
- net /EPD_DC: track 46.1 -> 98.2 mm
- net /EPD_MOSI: track 144.8 -> 131.3 mm
- net Net-(J1-Pin_2): track 8.31 -> 0.00 mm
- net GND: track 26.1 -> 29.9 mm
- net +3.3V: track 26.0 -> 26.4 mm, vias 3 -> 6
Other:
- outline, holes or cut-outs redrawn
- board text added: "BSY D5"
- board text added: "CS D2"
- board text added: "DC D3"
- board text added: "RST D4"
- board text removed: "BSY/D5"
- board text removed: "CS/D2"
- board text removed: "DC/D3"
- board text removed: "RST/D4"
